File: CAN-Interface-Board/LD0_3n3v.kicad_sch (KiCad schematic)
At the start: 3 parts, among them U2 LD1117S33TR

Commit message: altered connectors, layout refinement, added LEDS
Parts:
- C2: footprint Capacitor_SMD:C_1210_3225Metric_Pad1.33x2.70mm_HandSolder -> Capacitor_SMD:C_0805_2012Metric_Pad1.18x1.45mm_HandSolder; LCSC Part (none) -> C49678; lcsc C6565120 -> (none)
- C3: footprint Capacitor_SMD:C_01005_0402Metric_Pad0.57x0.30mm_HandSolder -> Capacitor_SMD:C_0805_2012Metric_Pad1.18x1.45mm_HandSolder; LCSC Part (none) -> C15850; lcsc C426118 -> (none)
- U2: LCSC Part (none) -> C86781; lcsc C86781 -> (none)
Changed lines of the file:
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@@
 			)
 		)
-		(property "Footprint" "Capacitor_SMD:C_01005_0402Metric_Pad0.57x0.30mm_HandSolder"
+		(property "Footprint" "Capacitor_SMD:C_0805_2012Metric_Pad1.18x1.45mm_HandSolder"
 			(at 98.7552 100.33 0)
 			(effects
@@
 			)
 		)
-		(property "lcsc" "C426118"
+		(property "LCSC Part" "C15850"
 			(at 97.79 96.52 0)
 			(effects
@@
 			)
 		)
-		(property "lcsc" "C86781"
+		(property "LCSC Part" "C86781"
 			(at 114.3 88.9 0)
 			(effects
@@
 			)
 		)
-		(property "Footprint" "Capacitor_SMD:C_1210_3225Metric_Pad1.33x2.70mm_HandSolder"
+		(property "Footprint" "Capacitor_SMD:C_0805_2012Metric_Pad1.18x1.45mm_HandSolder"
 			(at 127.9652 100.33 0)
 			(effects
@@
 			)
 		)
-		(property "lcsc" "C6565120"
+		(property "LCSC Part" "C49678"
 			(at 127 96.52 0)
 			(effects
