File: CAN-Interface-Board/CAN-Interface-Board.kicad_pcb (KiCad board)
At the start: 2 copper layers, 70 x 89 mm, 57 parts, among them CN1 Limit Switch Connector 1, CN2 Limit Switch Connector 2, CN3 Encoder Connector, CN5 XY-B3B-XH-A, CN6 MOLEX_26013114, CN7 MOLEX_CAN_IN, CN8 MOLEX_CAN_OUT, J1 USB_C_Receptacle, J2 Conn_01x04_Pin, J3 Conn_01x05_Pin, J4 Conn_01x04_Pin, Q1 INA180A2, U1 SN65HVD230, U2 LD1117S33TR, U3 STM32F405RGTx

Commit message: editing schematic
Parts:
- removed J3: Conn_01x05_Pin, Connector_PinHeader_2.54mm:PinHeader_1x05_P2.54mm_Vertical
- removed the REF** at (170.5, 126.0)
- removed the REF** at (112.0, 49.0)
- removed the REF** at (170.0, 49.0)
- removed the REF** at (112.5, 126.0)
- added REF**: MountingHole_3.2mm_M3_Pad_Via, MountingHole:MountingHole_3.2mm_M3_Pad_Via, F.Cu at (160.0, 41.0)
- added REF**: MountingHole_3.2mm_M3_Pad_Via, MountingHole:MountingHole_3.2mm_M3_Pad_Via, F.Cu at (121.0, 41.0)
- added REF**: MountingHole_3.2mm_M3_Pad_Via, MountingHole:MountingHole_3.2mm_M3_Pad_Via, F.Cu at (161.0, 131.0)
- added REF**: MountingHole_3.2mm_M3_Pad_Via, MountingHole:MountingHole_3.2mm_M3_Pad_Via, F.Cu at (121.0, 131.0)
- moved C19 105.2 mm to (253.7, 93.7)
- moved CN5 105.2 mm to (277.6, 73.0)
- moved D3 105.2 mm to (254.5, 88.5)
- moved J_BUCK_OUT_A1 105.2 mm to (262.5, 117.4)
- moved J_BUCK_OUT_B1 105.2 mm to (262.5, 102.9)
- moved R6 105.2 mm to (250.2, 93.7)
- moved CN6 105.2 mm to (225.1, 55.9)
- moved C1 105.2 mm to (253.0, 74.2)
- moved C10 105.2 mm to (244.6, 81.2)
- moved C11 105.2 mm to (241.1, 93.2)
- moved C12 105.2 mm to (232.6, 92.2)
- moved C13 105.2 mm to (227.1, 81.2)
- moved C14 105.2 mm to (245.1, 76.7)
- moved C15 105.2 mm to (232.1, 74.2)
- moved C16 105.2 mm to (227.1, 85.7)
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Other:
- board size 70 x 89 mm -> 165.1 x 100 mm
- copper layers 2 -> 4
