File: CAN-Interface-Board/CAN-Transciever.kicad_sch (KiCad schematic)
At the start: 4 parts, among them U1 SN65HVD230

Commit message: altered connectors, layout refinement, added LEDS
Parts:
- C1: footprint Capacitor_SMD:C_1210_3225Metric_Pad1.33x2.70mm_HandSolder -> Capacitor_SMD:C_0805_2012Metric_Pad1.18x1.45mm_HandSolder; LCSC Part (none) -> C49678; lcsc C6565120 -> (none)
- R1: LCSC Part (none) -> C4353191; lcsc C4353191 -> (none)
- U1: LCSC Part (none) -> C12084; lcsc C12084 -> (none)
Changed lines of the file:
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@@
 			)
 		)
-		(property "Footprint" "Capacitor_SMD:C_1210_3225Metric_Pad1.33x2.70mm_HandSolder"
+		(property "Footprint" "Capacitor_SMD:C_0805_2012Metric_Pad1.18x1.45mm_HandSolder"
 			(at 87.3252 110.49 0)
 			(effects
@@
 			)
 		)
-		(property "lcsc" "C6565120"
+		(property "LCSC Part" "C49678"
 			(at 86.36 106.68 0)
 			(effects
@@
 			)
 		)
-		(property "lcsc" "C4353191"
+		(property "LCSC Part" "C4353191"
 			(at 140.97 106.68 0)
 			(effects
@@
 			)
 		)
-		(property "lcsc" "C12084"
+		(property "LCSC Part" "C12084"
 			(at 125.73 105.41 0)
 			(effects

Commit message: editing schematic
Parts:
- removed C1: 100nF, Capacitor_SMD:C_0805_2012Metric_Pad1.18x1.45mm_HandSolder, symbol Device:C
- removed JP1: SolderJumper_2_Open, Jumper:SolderJumper-2_P1.3mm_Open_TrianglePad1.0x1.5mm, symbol Jumper:SolderJumper_2_Open
- removed R1: 120R, Resistor_SMD:R_0603_1608Metric, symbol Device:R
- removed U1: SN65HVD230, Package_SO:SOIC-8_3.9x4.9mm_P1.27mm, symbol Interface_CAN_LIN:SN65HVD230
- added C24: 100nf, Capacitor_SMD:C_0805_2012Metric_Pad1.18x1.45mm_HandSolder, symbol Device:C
- added CAN_IN1, CAN_OUT1: CAN, myFootprints:MOLEX_26013114, symbol Connector_Generic:Conn_01x02
- added JP2: SolderJumper_2_Open, Jumper:SolderJumper-2_P1.3mm_Open_TrianglePad1.0x1.5mm, symbol Jumper:SolderJumper_2_Open
- added R9: 120R, Resistor_SMD:R_0805_2012Metric_Pad1.20x1.40mm_HandSolder, symbol Device:R
- added U5: SN65HVD230, Package_SO:SOIC-8_3.9x4.9mm_P1.27mm, symbol Interface_CAN_LIN:SN65HVD230
Connections:
- net +3.3V: now also C24.1, U5.3 (VCC)
- net CANH: now also CAN_IN1.1 (Pin_1), CAN_OUT1.1 (Pin_1), R9.1, U5.7 (CANH)
- net CANL: now also CAN_IN1.2 (Pin_2), CAN_OUT1.2 (Pin_2), JP2.2 (B), U5.6 (CANL)
- net GND: now also C24.2, U5.2 (GND), U5.8 (Rs)
- new net: JP2.1 (A), R9.2
- new net CAN_RX_2: U5.4 (R)
- new net CAN_TX_2: U5.1 (D)
