File: CAN-Interface-Board/Current_Sensor.kicad_sch (KiCad schematic)
At the start: 4 parts, among them Q1 INA180A2

Commit message: altered connectors, layout refinement, added LEDS
Parts:
- C4, C5: footprint Capacitor_SMD:C_1210_3225Metric_Pad1.33x2.70mm_HandSolder -> Capacitor_SMD:C_0805_2012Metric_Pad1.18x1.45mm_HandSolder; LCSC Part (none) -> C49678; lcsc C6565120 -> (none)
- R4: footprint (none) -> Resistor_SMD:R_1206_3216Metric; LCSC Part (none) -> C4293416; lcsc C4293416 -> (none)
Changed lines of the file:
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@@
 			)
 		)
-		(property "Footprint" "Capacitor_SMD:C_1210_3225Metric_Pad1.33x2.70mm_HandSolder"
+		(property "Footprint" "Capacitor_SMD:C_0805_2012Metric_Pad1.18x1.45mm_HandSolder"
 			(at 115.2652 81.28 0)
 			(effects
@@
 			)
 		)
-		(property "lcsc" "C6565120"
+		(property "LCSC Part" "C49678"
 			(at 114.3 77.47 0)
 			(effects
@@
 			)
 		)
-		(property "Footprint" "Capacitor_SMD:C_1210_3225Metric_Pad1.33x2.70mm_HandSolder"
+		(property "Footprint" "Capacitor_SMD:C_0805_2012Metric_Pad1.18x1.45mm_HandSolder"
 			(at 146.05 62.5348 0)
 			(effects
@@
 			)
 		)
-		(property "lcsc" "C6565120"
+		(property "LCSC Part" "C49678"
 			(at 142.24 63.5 90)
 			(effects
@@
 			)
 		)
-		(property "Footprint" ""
+		(property "Footprint" "Resistor_SMD:R_1206_3216Metric"
 			(at 93.472 78.74 90)
 			(effects
@@
 			)
 		)
-		(property "lcsc" "C4293416"
+		(property "LCSC Part" "C4293416"
 			(at 95.25 78.74 0)
 			(effects

Commit message: editing schematic
Parts:
- R4: value 0.015Ohm -> 150r
Connections:
- net V-buck-out is gone; now on net +5V: C4.2, Q1.4 (-), R4.2
- net Signal renamed VoltageADC
- net V-buck-in renamed +5V
Other:
- moved on the sheet: C4, C5, Q1, R4
