File: Schematics/Barometer.kicad_sch (KiCad schematic)
At the start: 4 parts

Commit message: finished and ERC schematic
Parts:
- C21: renamed from C18; LCSC (none) -> C49678
- C22: renamed from C20; LCSC (none) -> C49678
- C23: renamed from C21; LCSC (none) -> C49678
- U4: renamed from U; LCSC (none) -> C54429
Connections:
- net BarometerSDL renamed BarometerSDA
Changed lines of the file:
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@@
 		)
 	)
-	(hierarchical_label "BarometerSDL"
+	(hierarchical_label "BarometerSDA"
 		(shape input)
 		(at 170.18 101.6 0)
@@
 		(dnp no)
 		(fields_autoplaced yes)
-		(property "Reference" "#PWR023"
+		(property "Reference" "#PWR068"
 			(at 107.95 115.57 0)
 			(effects
@@
 			(project "CAN-Interface-Board"
 				(path "/8a3e7f99-4046-40e8-bd7c-d9d1c8c7162e/a39ea6c8-c4df-4a74-9922-1f41a5f54a02"
-					(reference "#PWR023")
+					(reference "#PWR068")
 					(unit 1)
 				)
@@
 		(dnp no)
 		(fields_autoplaced yes)
-		(property "Reference" "U"
+		(property "Reference" "U4"
 			(at 153.035 92.71 0)
 			(effects
@@
 		)
 		(property "Footprint" "myFootprints:PSON80P300X300X100-8N"
-			(at 148.59 105.41 0)
+			(at 152.908 113.284 0)
 			(effects
 				(font
@@
 		)
 		(property "LCSC Part" "C54429"
+			(at 153.924 115.824 0)
+			(effects
+				(font
+					(size 1.27 1.27)
+				)
+				(hide yes)
+			)
+		)
+		(property "LCSC" "C54429"
 			(at 148.59 105.41 0)
 			(effects
@@
 			(project "CAN-Interface-Board"
 				(path "/8a3e7f99-4046-40e8-bd7c-d9d1c8c7162e/a39ea6c8-c4df-4a74-9922-1f41a5f54a02"
-					(reference "U")
+					(reference "U4")
 					(unit 1)
 				)
@@
 		(dnp no)
 		(fields_autoplaced yes)
-		(property "Reference" "#PWR024"
+		(property "Reference" "#PWR069"
 			(at 143.51 105.41 0)
 			(effects
@@
 			(project "CAN-Interface-Board"
 				(path "/8a3e7f99-4046-40e8-bd7c-d9d1c8c7162e/a39ea6c8-c4df-4a74-9922-1f41a5f54a02"
-					(reference "#PWR024")
+					(reference "#PWR069")
 					(unit 1)
 				)
@@
 		(on_board yes)
 		(dnp no)
-		(property "Reference" "C18"
+		(property "Reference" "C21"
 			(at 115.57 102.8699 0)
 			(effects
@@
 			)
 		)
+		(property "LCSC" "C49678"
+			(at 111.76 104.14 0)
+			(effects
+				(font
+					(size 1.27 1.27)
+				)
+				(hide yes)
+			)
+		)
 		(pin "1"
 		)
@@
 			(project "CAN-Interface-Board"
 				(path "/8a3e7f99-4046-40e8-bd7c-d9d1c8c7162e/a39ea6c8-c4df-4a74-9922-1f41a5f54a02"
-					(reference "C18")
+					(reference "C21")
 					(unit 1)
 				)
@@
 		(on_board yes)
 		(dnp no)
-		(property "Reference" "C20"
+		(property "Reference" "C22"
 			(at 125.73 102.8699 0)
 			(effects
@@
 			)
 		)
+		(property "LCSC" "C49678"
+			(at 121.92 104.14 0)
+			(effects
+				(font
+					(size 1.27 1.27)
+				)
+				(hide yes)
+			)
+		)
 		(pin "1"
 		)
@@
 			(project "CAN-Interface-Board"
 				(path "/8a3e7f99-4046-40e8-bd7c-d9d1c8c7162e/a39ea6c8-c4df-4a74-9922-1f41a5f54a02"
-					(reference "C20")
+					(reference "C22")
 					(unit 1)
 				)
@@
 		(dnp no)
 		(fields_autoplaced yes)
-		(property "Reference" "#PWR022"
+		(property "Reference" "#PWR067"
 			(at 107.95 102.87 0)
 			(effects
@@
 			(project "CAN-Interface-Board"
 				(path "/8a3e7f99-4046-40e8-bd7c-d9d1c8c7162e/a39ea6c8-c4df-4a74-9922-1f41a5f54a02"
-					(reference "#PWR022")
+					(reference "#PWR067")
 					(unit 1)
 				)
@@
 		(on_board yes)
 		(dnp no)
-		(property "Reference" "C21"
+		(property "Reference" "C23"
 			(at 134.62 104.1399 0)
 			(effects
@@
 			)
 		)
+		(property "LCSC" "C49678"
+			(at 130.81 105.41 0)
+			(effects
+				(font
+					(size 1.27 1.27)
+				)
+				(hide yes)
+			)
+		)
 		(pin "1"
 		)
@@
 			(project "CAN-Interface-Board"
 				(path "/8a3e7f99-4046-40e8-bd7c-d9d1c8c7162e/a39ea6c8-c4df-4a74-9922-1f41a5f54a02"
-					(reference "C21")
-					(unit 1)
-				)
+					(reference "C23")
+					(unit 1)
+				)
