File: Schematics/CAN-Transciever.kicad_sch (KiCad schematic)
At the start: 6 parts, among them U5 SN65HVD230

Commit message: finished and ERC schematic
Parts:
- C3: renamed from C24; LCSC (none) -> C49678
- CAN_IN1, CAN_OUT1: LCSC (none) -> C17644051
- R2: renamed from R9; value 120R -> 120r; LCSC (none) -> C269726
- U1: renamed from U5; LCSC (none) -> C1543812
- renumbered JP2 to JP1
Changed lines of the file:
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@@
 			)
 		)
-		(property "Package" ""
-			(at 190.5 86.36 0)
-			(effects
-				(font
-					(size 1.27 1.27)
-				)
-				(hide yes)
-			)
-		)
-		(property "Price" ""
-			(at 190.5 86.36 0)
-			(effects
-				(font
-					(size 1.27 1.27)
-				)
-				(hide yes)
-			)
-		)
-		(property "Purchase-URL" ""
+		(property "LCSC" "C17644051"
 			(at 190.5 86.36 0)
 			(effects
@@
 		(dnp no)
 		(fields_autoplaced yes)
-		(property "Reference" "R9"
+		(property "Reference" "R2"
 			(at 151.13 90.1699 0)
 			(effects
@@
 			)
 		)
-		(property "Value" "120R"
+		(property "Value" "120r"
 			(at 151.13 92.7099 0)
 			(effects
@@
 			)
 		)
-		(property "Package" ""
+		(property "LCSC" "C269726"
 			(at 148.59 91.44 0)
 			(effects
@@
 			)
 		)
-		(property "Price" ""
-			(at 148.59 91.44 0)
-			(effects
-				(font
-					(size 1.27 1.27)
-				)
-				(hide yes)
-			)
-		)
-		(property "Purchase-URL" ""
-			(at 148.59 91.44 0)
-			(effects
-				(font
-					(size 1.27 1.27)
-				)
-				(hide yes)
-			)
-		)
 		(pin "1"
 		)
@@
 			(project "CAN-Interface-Board"
 				(path "/8a3e7f99-4046-40e8-bd7c-d9d1c8c7162e/5582202c-f32a-4245-a5f8-7aec56821a23"
-					(reference "R9")
+					(reference "R2")
 					(unit 1)
 				)
@@
 		(dnp no)
 		(fields_autoplaced yes)
-		(property "Reference" "#PWR038"
+		(property "Reference" "#PWR07"
 			(at 133.35 78.74 0)
 			(effects
@@
 			(project "CAN-Interface-Board"
 				(path "/8a3e7f99-4046-40e8-bd7c-d9d1c8c7162e/5582202c-f32a-4245-a5f8-7aec56821a23"
-					(reference "#PWR038")
+					(reference "#PWR07")
 					(unit 1)
 				)
@@
 		(dnp no)
 		(fields_autoplaced yes)
-		(property "Reference" "#PWR037"
+		(property "Reference" "#PWR06"
 			(at 114.3 95.25 0)
 			(effects
@@
 			(project "CAN-Interface-Board"
 				(path "/8a3e7f99-4046-40e8-bd7c-d9d1c8c7162e/5582202c-f32a-4245-a5f8-7aec56821a23"
-					(reference "#PWR037")
+					(reference "#PWR06")
 					(unit 1)
 				)
@@
 		(on_board yes)
 		(dnp no)
-		(property "Reference" "C24"
+		(property "Reference" "C3"
 			(at 97.79 90.1699 0)
 			(effects
@@
 			)
 		)
-		(property "Package" ""
+		(property "LCSC" "C49678"
 			(at 93.98 91.44 0)
 			(effects
@@
 			)
 		)
-		(property "Price" ""
-			(at 93.98 91.44 0)
-			(effects
-				(font
-					(size 1.27 1.27)
-				)
-				(hide yes)
-			)
-		)
-		(property "Purchase-URL" ""
-			(at 93.98 91.44 0)
-			(effects
-				(font
-					(size 1.27 1.27)
-				)
-				(hide yes)
-			)
-		)
 		(pin "1"
 		)
@@
 			(project "CAN-Interface-Board"
 				(path "/8a3e7f99-4046-40e8-bd7c-d9d1c8c7162e/5582202c-f32a-4245-a5f8-7aec56821a23"
-					(reference "C24")
+					(reference "C3")
 					(unit 1)
 				)
@@
 		(on_board yes)
 		(dnp no)
-		(property "Reference" "JP2"
+		(property "Reference" "JP1"
 			(at 153.67 102.616 0)
 			(effects
@@
 			)
 		)
-		(property "Package" ""
-			(at 153.67 95.25 0)
-			(effects
-				(font
-					(size 1.27 1.27)
-				)
-				(hide yes)
-			)
-		)
-		(property "Price" ""
-			(at 153.67 95.25 0)
-			(effects
-				(font
-					(size 1.27 1.27)
-				)
-				(hide yes)
-			)
-		)
-		(property "Purchase-URL" ""
-			(at 153.67 95.25 0)
-			(effects
-				(font
-					(size 1.27 1.27)
-				)
-				(hide yes)
-			)
-		)
 		(pin "1"
 		)
@@
 			(project "CAN-Interface-Board"
 				(path "/8a3e7f99-4046-40e8-bd7c-d9d1c8c7162e/5582202c-f32a-4245-a5f8-7aec56821a23"
-					(reference "JP2")
+					(reference "JP1")
 					(unit 1)
 				)
@@
 			)
 		)
-		(property "Package" ""
-			(at 190.5 95.25 0)
-			(effects
-				(font
-					(size 1.27 1.27)
-				)
-				(hide yes)
-			)
-		)
-		(property "Price" ""
-			(at 190.5 95.25 0)
-			(effects
-				(font
-					(size 1.27 1.27)
-				)
-				(hide yes)
-			)
-		)
-		(property "Purchase-URL" ""
+		(property "LCSC" "C17644051"
 			(at 190.5 95.25 0)
 			(effects
@@
 		(dnp no)
 		(fields_autoplaced yes)
-		(property "Reference" "#PWR039"
+		(property "Reference" "#PWR08"
 			(at 133.35 113.03 0)
 			(effects
@@
 			(project "CAN-Interface-Board"
 				(path "/8a3e7f99-4046-40e8-bd7c-d9d1c8c7162e/5582202c-f32a-4245-a5f8-7aec56821a23"
-					(reference "#PWR039")
+					(reference "#PWR08")
 					(unit 1)
 				)
@@
 		(dnp no)
 		(fields_autoplaced yes)
-		(property "Reference" "U5"
+		(property "Reference" "U1"
 			(at 135.4933 80.01 0)
 			(effects
@@
 			)
 		)
-		(property "Package" ""
+		(property "LCSC" "C1543812"
 			(at 133.35 90.17 0)
 			(effects
@@
 			)
 		)
-		(property "Price" ""
-			(at 133.35 90.17 0)
-			(effects
-				(font
-					(size 1.27 1.27)
-				)
-				(hide yes)
-			)
-		)
-		(property "Purchase-URL" ""
-			(at 133.35 90.17 0)
-			(effects
-				(font
-					(size 1.27 1.27)
-				)
-				(hide yes)
-			)
-		)
 		(pin "1"
 		)
@@
 			(project "CAN-Interface-Board"
 				(path "/8a3e7f99-4046-40e8-bd7c-d9d1c8c7162e/5582202c-f32a-4245-a5f8-7aec56821a23"
-					(reference "U5")
-					(unit 1)
-				)
+					(reference "U1")
+					(unit 1)
+				)
