File: Schematics/FlashSD.kicad_sch (KiCad schematic)
At the start: 4 parts, among them J8 Micro_SD_Card

Commit message: finished and ERC schematic
Parts:
- removed D2: SRV05-4.TCT, myFootprints:SOT95P280X145-6N, symbol SRV05-4.TCT:SRV05-4.TCT
- J3: renamed from J8; LCSC (none) -> C164170
- R8: renamed from R17; value 220R -> 33r; LCSC (none) -> C126353
- R9: renamed from R16; LCSC (none) -> C84376
Connections:
- no-connect marks 4 -> 2
Other:
- moved on the sheet: R8
