File: Schematics/Power.kicad_sch (KiCad schematic)
At the start: 10 parts, among them U2 LDL1117-3.3

Commit message: finished and ERC schematic
Parts:
- C4: renamed from C2; LCSC (none) -> C28323
- C5: renamed from C3; LCSC (none) -> C98192
- D1: renamed from D6; LCSC (none) -> C113936
- D2: renamed from D7; LCSC (none) -> C113936
- J_BUCK_IN_A1: renamed from J_BUCK_IN_A2; now in the parts list
- J_BUCK_IN_B1: renamed from J_BUCK_IN_B2; now in the parts list
- J_BUCK_OUT_A1: renamed from J_BUCK_OUT_A2; now in the parts list
- J_BUCK_OUT_B1: renamed from J_BUCK_OUT_B2; now in the parts list
- U2: LCSC (none) -> C435835
