File: Schematics/MCU.kicad_sch (KiCad schematic)
At the start: 30 parts, among them J2 Conn_01x04_Pin, J3 Microsemi_FlashPro-JTAG-10, J4 Conn_01x03_Pin, J5 Conn_01x03_Pin, U3 STM32F405RGTx, Y1 8mhz

Commit message: finished and ERC schematic
Parts:
- removed J2: Conn_01x04_Pin, Connector_PinHeader_2.54mm:PinHeader_1x04_P2.54mm_Vertical, symbol Connector:Conn_01x04_Pin
- removed J4, J5: Conn_01x03_Pin, symbol Connector:Conn_01x03_Pin
- BootSwitch1: renamed from BootSwitch2; LCSC (none) -> C49393646
- C10: renamed from C11; LCSC (none) -> C49678
- C11: renamed from C12; LCSC (none) -> C49678
- C12: renamed from C13; LCSC (none) -> C49678
- C13: renamed from C7; LCSC (none) -> C28323
- C14: renamed from C8; LCSC (none) -> C49678
- C15: renamed from C14; LCSC (none) -> C49678
- C16: renamed from C15; LCSC (none) -> C49678
- C17: renamed from C16; LCSC (none) -> C28323
- C18: renamed from C17; LCSC (none) -> C49678
- C19: renamed from C1; LCSC (none) -> C170109
- C20: renamed from C25; LCSC (none) -> C170109
- C6: renamed from C27; LCSC (none) -> C49678
- C7: renamed from C28; LCSC (none) -> C49678
- C8: renamed from C9; LCSC (none) -> C19110
- C9: renamed from C10; LCSC (none) -> C19110
- CBulk1: LCSC (none) -> C98192
- D3: renamed from D4; LCSC (none) -> C2827321
- FB1: LCSC (none) -> C85840
- J1: renamed from J3; LCSC (none) -> C585350
- PowerLED1: renamed from PowerLED2; LCSC (none) -> C965799
- R3: renamed from R2; LCSC (none) -> C84376
- R4: renamed from R2; LCSC (none) -> C96346
- R5: renamed from R3; LCSC (none) -> C95781
- RSTSwitch1: LCSC (none) -> C49393646
- U3: value STM32F405RGTx -> STM32F405RGT6; LCSC (none) -> C15742
- Y1: LCSC (none) -> C19723344
Connections:
- net OSC IN: now also U3.5 (PH0)
- net OSC OUT: now also U3.6 (PH1)
- net SPI2_MISO: now reaches U3.10 (PC2)
- net SPI2_MOSI: now reaches U3.11 (PC3)
- net CS_IMU: now reaches U3.20 (PA4)
- net SPI1_MISO: now reaches U3.22 (PA6)
- net PWMServo_Roll: now reaches U3.26 (PB0)
- net PWMServo_CAS: now reaches U3.27 (PB1)
- net 5Venable: now reaches U3.28 (PB2)
- net SPI2_SCK: now reaches U3.29 (PB10)
- net IMU_Interrutpt: now reaches U3.55 (PB3)
- net LimitSwitchCAS: now reaches U3.56 (PB4)
- net LimitSwitchRoll: now reaches U3.57 (PB5)
- net I2C_SCL: now reaches U3.58 (PB6)
- net I2C_SDA: now reaches U3.59 (PB7)
- net CAN_RS renamed SPI1_SCK
- net ENCODER_A: no longer names the net of U3.14 (PA0)
- net ENCODER_B: no longer names the net of U3.15 (PA1)
- net Servo_Signal renamed SPI1_MOSI
- no-connect marks 40 -> 34

Commit message: inital layout started, refining stage
Parts:
- removed CBulk1: 4.7u, Capacitor_SMD:C_0805_2012Metric_Pad1.18x1.45mm_HandSolder, symbol Device:C
- added C30: 4.7u, Capacitor_SMD:C_0805_2012Metric_Pad1.18x1.45mm_HandSolder, symbol Device:C
Connections:
- net +3.3V: now also C30.1; no longer C14.2, C17.1, C18.1, FB1.2, U3.13 (VDDA)
- net GND: now also C30.2
- new net +3.3VA: C14.2, C17.1, C18.1, FB1.2, U3.13 (VDDA)
Other:
- moved on the sheet: C10, C17, C18
