File: Schematics/Servo.kicad_sch (KiCad schematic)
At the start: 5 parts, among them CN4 XY-B3B-XH-A, CN5 Limit Switch Connector 1, CN6 Limit Switch Connector 2

Commit message: finished and ERC schematic
Parts:
- added C26, C28: 1uf, Capacitor_SMD:C_0805_2012Metric_Pad1.18x1.45mm_HandSolder, symbol Device:C
- added C27: 100nf, Capacitor_SMD:C_0805_2012Metric_Pad1.18x1.45mm_HandSolder, symbol Device:C
- added C29: 47uf, Capacitor_SMD:C_0805_2012Metric_Pad1.18x1.45mm_HandSolder, symbol Device:C
- added CN3: XY-B3B-XH-A, custom footprints:CONN-TH_3P-P2.50_A2501WV2-3P, symbol custom symbols:XY-B3B-XH-A
- added R11: 100k, Resistor_SMD:R_0805_2012Metric_Pad1.20x1.40mm_HandSolder, symbol Device:R
- added U6: TPS22917DBVR, myFootprints:SOT95P280X145-6N, symbol TPS22917DBVR:TPS22917DBVR
- CN1: renamed from CN5; LCSC (none) -> C158012; Manufacturer Part B2B-XH-A(LF)(SN) -> (none); Supplier LCSC -> (none)
- CN2: renamed from CN6; LCSC (none) -> C158012; Manufacturer Part B2B-XH-A(LF)(SN) -> (none); Supplier LCSC -> (none)
- CN4: LCSC (none) -> C51940188; Manufacturer Part XY-B3B-XH-A -> (none)
- R12: renamed from R1; value 10K -> 10k; LCSC (none) -> C84376
- R13: renamed from R10; value 10K -> 10k; LCSC (none) -> C84376
Connections:
- net +3.3V: now also R11.2
- net GND: now also C26.2, C27.2, C28.2, C29.2, CN3.1, U6.2 (GND)
- net Limit_Switch_A renamed Limit_Switch_CAS
- net Limit_Switch_B renamed Limit_Switch_Roll
- net Servo_Signal renamed Servo_Airbrakes
- net Servo_VCC: no longer names the net of CN4.2
- net Servo_VCC: now also C27.1, C28.1, C29.1, CN3.2, U6.6 (VOUT)
- new net PWN_EN: R11.1, U6.3 (ON)
- new net Servo5V: C26.1, U6.1 (VIN)
- new net Servo_RollControl: CN3.3
- no-connect marks 0 -> 2
Other:
- moved on the sheet: CN1, CN2, CN4, R12, R13

Commit message: inital layout started, refining stage
Parts:
- CN1, CN2: footprint custom footprints:JST B2B-XH-A(LF)(SN) -> myFootprints:JST_B2B-XH-A_LF__SN_
- CN3, CN4: footprint custom footprints:CONN-TH_3P-P2.50_A2501WV2-3P -> myFootprints:JST_B3B-XH-A
Other:
- moved on the sheet: CN3
Changed lines of the file:
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@@
 	(wire
 		(pts
-			(xy 196.85 53.34) (xy 213.36 53.34)
+			(xy 196.85 53.34) (xy 215.9 53.34)
 		)
 		(stroke
@@
 	(wire
 		(pts
+			(xy 215.9 50.8) (xy 213.36 50.8)
+		)
+		(stroke
+			(width 0)
+			(type default)
+		)
+	)
+	(wire
+		(pts
 			(xy 172.72 58.42) (xy 160.02 58.42)
+		)
+		(stroke
+			(width 0)
+			(type default)
+		)
+	)
+	(wire
+		(pts
+			(xy 215.9 55.88) (xy 213.36 55.88)
 		)
 		(stroke
@@
 			)
 		)
-		(property "Footprint" "custom footprints:JST B2B-XH-A(LF)(SN)"
+		(property "Footprint" "myFootprints:JST_B2B-XH-A_LF__SN_"
 			(at 106.68 96.52 0)
 			(effects
@@
 	)
 	(symbol
+		(lib_name "XY-B3B-XH-A_1")
 		(lib_id "custom symbols:XY-B3B-XH-A")
-		(at 218.44 53.34 0)
+		(at 220.98 53.34 0)
 		(unit 1)
 		(exclude_from_sim no)
@@
 		(fields_autoplaced yes)
 		(property "Reference" "CN3"
-			(at 222.25 52.0699 0)
+			(at 224.79 52.0699 0)
 			(effects
 				(font
@@
 		)
 		(property "Value" "XY-B3B-XH-A"
-			(at 222.25 54.6099 0)
-			(effects
-				(font
-					(size 1.27 1.27)
-				)
-				(justify left)
-			)
-		)
-		(property "Footprint" "custom footprints:CONN-TH_3P-P2.50_A2501WV2-3P"
-			(at 218.44 53.34 0)
+			(at 224.79 54.6099 0)
+			(effects
+				(font
+					(size 1.27 1.27)
+				)
+				(justify left)
+			)
+		)
+		(property "Footprint" "myFootprints:JST_B3B-XH-A"
+			(at 222.25 62.992 0)
 			(effects
 				(font
@@
 		)
 		(property "Datasheet" ""
-			(at 218.44 53.34 0)
+			(at 220.98 53.34 0)
 			(effects
 				(font
@@
 		)
 		(property "Description" ""
-			(at 218.44 53.34 0)
+			(at 220.98 53.34 0)
 			(effects
 				(font
@@
 		)
 		(property "Manufacturer" "XYECONN(辛译)"
-			(at 228.6 53.34 0)
+			(at 237.998 66.294 0)
 			(effects
 				(font
@@
 		)
 		(property "LCSC Part" "C51940188"
-			(at 226.822 51.562 0)
+			(at 237.998 59.944 0)
 			(effects
 				(font
@@
 		)
 		(property "LCSC" "C51940188"
-			(at 218.44 53.34 0)
+			(at 220.726 66.294 0)
 			(effects
 				(font
@@
 			)
 		)
-		(property "Footprint" "custom footprints:JST B2B-XH-A(LF)(SN)"
+		(property "Footprint" "myFootprints:JST_B2B-XH-A_LF__SN_"
 			(at 177.8 95.25 0)
 			(effects
@@
 			)
 		)
-		(property "Footprint" "custom footprints:CONN-TH_3P-P2.50_A2501WV2-3P"
+		(property "Footprint" "myFootprints:JST_B3B-XH-A"
 			(at 218.44 67.31 0)
 			(effects
