File: Schematics/IMU.kicad_sch (KiCad schematic)
At the start: 4 parts, among them U4 LSM6DS3TR-C

Commit message: finished and ERC schematic
Parts:
- removed C26: 100nf, Capacitor_SMD:C_0805_2012Metric_Pad1.18x1.45mm_HandSolder, symbol Device:C
- added R10: 10k, Resistor_SMD:R_0805_2012Metric_Pad1.20x1.40mm_HandSolder, symbol Device:R
- C24: renamed from C22; LCSC (none) -> C49678
- C25: renamed from C23; LCSC (none) -> C49678
- U5: renamed from U4; LCSC (none) -> C967633
Connections:
- net +3.3V: now also R10.1; no longer U5.12 (CS)
- net GND: no longer U5.1 (SDO/SA0), U5.2 (SDx), U5.3 (SCx)
- net IMU_DReady: now reaches U5.9 (INT2)
- net IMUSCL renamed IMU_SCK
- net IMUSDA renamed IMU_MOSI
- new net: R10.2, U5.12 (CS)
- new net IMU_MISO: U5.1 (SDO/SA0)
- no-connect marks 2 -> 3
Other:
- note added: "Using SPI for faster reads for control"

Commit message: fixed schematic
Connections:
- net IMU_CS: now reaches R10.2, U5.12 (CS)
Other:
- moved on the sheet: R10
Changed lines of the file:
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@@
+	)
+	(junction
+		(at 139.7 76.2)
+		(diameter 0)
+		(color 0 0 0 0)
 	)
 	(junction
@@
 	)
 	(junction
-		(at 139.7 73.66)
-		(diameter 0)
-		(color 0 0 0 0)
-	)
-	(junction
 		(at 137.16 123.19)
 		(diameter 0)
@@
 	(wire
 		(pts
+			(xy 139.7 76.2) (xy 139.7 97.79)
+		)
+		(stroke
+			(width 0)
+			(type default)
+		)
+	)
+	(wire
+		(pts
 			(xy 115.57 113.03) (xy 125.73 113.03)
 		)
@@
 	(wire
 		(pts
-			(xy 154.94 73.66) (xy 139.7 73.66)
-		)
-		(stroke
-			(width 0)
-			(type default)
-		)
-	)
-	(wire
-		(pts
-			(xy 139.7 82.55) (xy 139.7 97.79)
+			(xy 139.7 73.66) (xy 139.7 76.2)
 		)
 		(stroke
@@
 	(wire
 		(pts
+			(xy 151.13 76.2) (xy 139.7 76.2)
+		)
+		(stroke
+			(width 0)
+			(type default)
+		)
+	)
+	(wire
+		(pts
 			(xy 142.24 82.55) (xy 149.86 82.55)
 		)
@@
 	(wire
 		(pts
-			(xy 139.7 73.66) (xy 139.7 74.93)
-		)
-		(stroke
-			(width 0)
-			(type default)
-		)
-	)
-	(wire
-		(pts
-			(xy 139.7 72.39) (xy 139.7 73.66)
+			(xy 139.7 63.5) (xy 139.7 66.04)
 		)
 		(stroke
@@
 	(hierarchical_label "IMU_CS"
 		(shape input)
-		(at 154.94 73.66 0)
+		(at 151.13 76.2 0)
 		(effects
 			(font
@@
 	(symbol
 		(lib_id "power:+3.3V")
-		(at 139.7 72.39 90)
+		(at 139.7 63.5 90)
 		(unit 1)
 		(exclude_from_sim no)
@@
 		(fields_autoplaced yes)
 		(property "Reference" "#PWR073"
-			(at 143.51 72.39 0)
+			(at 143.51 63.5 0)
 			(effects
 				(font
@@
 		)
 		(property "Value" "+3.3V"
-			(at 135.89 72.3899 90)
+			(at 135.89 63.4999 90)
 			(effects
 				(font
@@
 		)
 		(property "Footprint" ""
-			(at 139.7 72.39 0)
+			(at 139.7 63.5 0)
 			(effects
 				(font
@@
 		)
 		(property "Datasheet" ""
-			(at 139.7 72.39 0)
+			(at 139.7 63.5 0)
 			(effects
 				(font
@@
 		)
 		(property "Description" "Power symbol creates a global label with name \"+3.3V\""
-			(at 139.7 72.39 0)
+			(at 139.7 63.5 0)
 			(effects
 				(font
@@
 	(symbol
 		(lib_id "Device:R")
-		(at 139.7 78.74 0)
+		(at 139.7 69.85 0)
 		(unit 1)
 		(exclude_from_sim no)
@@
 		(fields_autoplaced yes)
 		(property "Reference" "R10"
-			(at 142.24 77.4699 0)
+			(at 142.24 68.5799 0)
 			(effects
 				(font
@@
 		)
 		(property "Value" "10k"
-			(at 142.24 80.0099 0)
+			(at 142.24 71.1199 0)
 			(effects
 				(font
@@
 		)
 		(property "Footprint" "Resistor_SMD:R_0805_2012Metric_Pad1.20x1.40mm_HandSolder"
-			(at 137.922 78.74 90)
+			(at 137.922 69.85 90)
 			(effects
 				(font
@@
 		)
 		(property "Datasheet" "~"
-			(at 139.7 78.74 0)
+			(at 139.7 69.85 0)
 			(effects
 				(font
@@
 		)
 		(property "Description" "Resistor"
-			(at 139.7 78.74 0)
+			(at 139.7 69.85 0)
 			(effects
 				(font
@@
 		)
 		(property "LCSC" "C84376"
-			(at 139.7 78.74 0)
-			(effects
-				(font
+			(at 139.7 69.85 0)
+			(effects
+				(font
