File: Schematics/usb_type_c.kicad_sch (KiCad schematic)
At the start: 4 parts, among them J1 USB_C_Receptacle

Commit message: finished and ERC schematic
Parts:
- D4: renamed from D1; LCSC (none) -> C13612; Package None -> (none); Price None -> (none); SnapEDA_Link https://www.snapeda.com/parts/SRV05-4.TCT/UMW/view-part/?re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 -> (none)
- J2: renamed from J1; LCSC (none) -> C49566391
- R6: renamed from R7; LCSC (none) -> C27834
- R7: renamed from R8; LCSC (none) -> C27834
Connections:
- net +5V: no longer J2.A4 (VBUS), J2.A9 (VBUS), J2.B4 (VBUS), J2.B9 (VBUS)
- new net USB5V: J2.A4 (VBUS), J2.A9 (VBUS), J2.B4 (VBUS), J2.B9 (VBUS)
Changed lines of the file:
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@@
+		)
+	)
+	(hierarchical_label "USB5V"
+		(shape output)
+		(at 115.57 71.12 0)
+		(effects
+			(font
+				(size 1.27 1.27)
+			)
+			(justify left)
 		)
 	)
@@
 		(dnp no)
 		(fields_autoplaced yes)
-		(property "Reference" "J1"
+		(property "Reference" "J2"
 			(at 82.55 63.5 0)
 			(effects
@@
 			)
 		)
+		(property "LCSC" "C49566391"
+			(at 82.55 96.52 0)
+			(effects
+				(font
+					(size 1.27 1.27)
+				)
+				(hide yes)
+			)
+		)
 		(pin "S1"
 		)
@@
 			(project ""
 				(path "/8a3e7f99-4046-40e8-bd7c-d9d1c8c7162e/f33094e5-7720-4bb5-9ddf-b2cfd7a85122"
-					(reference "J1")
+					(reference "J2")
 					(unit 1)
 				)
@@
 		(on_board yes)
 		(dnp no)
-		(property "Reference" "#PWR0113"
+		(property "Reference" "#PWR060"
 			(at 135.89 85.09 0)
 			(effects
@@
 			(project "CAN-Interface-Board"
 				(path "/8a3e7f99-4046-40e8-bd7c-d9d1c8c7162e/f33094e5-7720-4bb5-9ddf-b2cfd7a85122"
-					(reference "#PWR0113")
-					(unit 1)
-				)
-			)
-		)
-	)
-	(symbol
-		(lib_id "power:+5V")
-		(at 115.57 71.12 270)
-		(unit 1)
-		(exclude_from_sim no)
-		(in_bom yes)
-		(on_board yes)
-		(dnp no)
-		(fields_autoplaced yes)
-		(property "Reference" "#PWR0117"
-			(at 111.76 71.12 0)
-			(effects
-				(font
-					(size 1.27 1.27)
-				)
-				(hide yes)
-			)
-		)
-		(property "Value" "+5V"
-			(at 119.38 71.1199 90)
-			(effects
-				(font
-					(size 1.27 1.27)
-				)
-				(justify left)
-			)
-		)
-		(property "Footprint" ""
-			(at 115.57 71.12 0)
-			(effects
-				(font
-					(size 1.27 1.27)
-				)
-				(hide yes)
-			)
-		)
-		(property "Datasheet" ""
-			(at 115.57 71.12 0)
-			(effects
-				(font
-					(size 1.27 1.27)
-				)
-				(hide yes)
-			)
-		)
-		(property "Description" "Power symbol creates a global label with name \"+5V\""
-			(at 115.57 71.12 0)
-			(effects
-				(font
-					(size 1.27 1.27)
-				)
-				(hide yes)
-			)
-		)
-		(pin "1"
-		)
-		(instances
-			(project ""
-				(path "/65068a32-f105-4204-b50e-234054c5a6d0/880da092-1c6b-4dcf-a509-490b22fc0ebc"
-					(reference "#PWR050")
-					(unit 1)
-				)
-			)
-			(project "CAN-Interface-Board"
-				(path "/8a3e7f99-4046-40e8-bd7c-d9d1c8c7162e/f33094e5-7720-4bb5-9ddf-b2cfd7a85122"
-					(reference "#PWR0117")
+					(reference "#PWR060")
 					(unit 1)
 				)
@@
 		(dnp no)
 		(fields_autoplaced yes)
-		(property "Reference" "D1"
+		(property "Reference" "D4"
 			(at 127 95.25 0)
 			(effects
@@
 			)
 		)
-		(property "Price" "None"
-			(at 137.16 87.63 0)
-			(effects
-				(font
-					(size 1.27 1.27)
-				)
-				(justify bottom)
-				(hide yes)
-			)
-		)
-		(property "Package" "None"
-			(at 137.16 87.63 0)
-			(effects
-				(font
-					(size 1.27 1.27)
-				)
-				(justify bottom)
-				(hide yes)
-			)
-		)
 		(property "Check_prices" "https://www.snapeda.com/parts/SRV05-4.TCT/UMW/view-part/?ref=eda"
 			(at 137.16 87.63 0)
@@
 			)
 		)
-		(property "SnapEDA_Link" "https://www.snapeda.com/parts/SRV05-4.TCT/UMW/view-part/?ref=snap"
-			(at 137.16 87.63 0)
-			(effects
-				(font
-					(size 1.27 1.27)
-				)
-				(justify bottom)
-				(hide yes)
-			)
-		)
 		(property "MP" "SRV05-4.TCT"
 			(at 137.16 87.63 0)
@@
 				)
 				(justify bottom)
+				(hide yes)
+			)
+		)
+		(property "LCSC" "C13612"
+			(at 137.16 87.63 0)
+			(effects
+				(font
+					(size 1.27 1.27)
+				)
 				(hide yes)
 			)
@@
 			(project ""
 				(path "/8a3e7f99-4046-40e8-bd7c-d9d1c8c7162e/f33094e5-7720-4bb5-9ddf-b2cfd7a85122"
-					(reference "D1")
+					(reference "D4")
 					(unit 1)
 				)
@@
 		(dnp no)
 		(fields_autoplaced yes)
-		(property "Reference" "#PWR0114"
+		(property "Reference" "#PWR061"
 			(at 149.86 93.98 0)
 			(effects
@@
 			(project "CAN-Interface-Board"
 				(path "/8a3e7f99-4046-40e8-bd7c-d9d1c8c7162e/f33094e5-7720-4bb5-9ddf-b2cfd7a85122"
-					(reference "#PWR0114")
+					(reference "#PWR061")
 					(unit 1)
 				)
@@
 		(on_board yes)
 		(dnp no)
-		(property "Reference" "#PWR0115"
+		(property "Reference" "#PWR059"
 			(at 146.05 82.55 0)
 			(effects
@@
 			(project "CAN-Interface-Board"
 				(path "/8a3e7f99-4046-40e8-bd7c-d9d1c8c7162e/f33094e5-7720-4bb5-9ddf-b2cfd7a85122"
-					(reference "#PWR0115")
+					(reference "#PWR059")
 					(unit 1)
 				)
@@
 		(dnp no)
 		(fields_autoplaced yes)
-		(property "Reference" "#PWR0118"
+		(property "Reference" "#PWR058"
 			(at 78.74 148.59 0)
 			(effects
@@
 			(project "CAN-Interface-Board"
 				(path "/8a3e7f99-4046-40e8-bd7c-d9d1c8c7162e/f33094e5-7720-4bb5-9ddf-b2cfd7a85122"
-					(reference "#PWR0118")
+					(reference "#PWR058")
 					(unit 1)
 				)
@@
 		(dnp no)
 		(fields_autoplaced yes)
-		(property "Reference" "R7"
+		(property "Reference" "R6"
 			(at 152.4 81.2799 0)
 			(effects
@@
 			)
 		)
+		(property "LCSC" "C27834"
+			(at 149.86 82.55 0)
+			(effects
+				(font
+					(size 1.27 1.27)
+				)
+				(hide yes)
+			)
+		)
 		(pin "1"
 		)
@@
 			(project ""
 				(path "/8a3e7f99-4046-40e8-bd7c-d9d1c8c7162e/f33094e5-7720-4bb5-9ddf-b2cfd7a85122"
-					(reference "R7")
+					(reference "R6")
 					(unit 1)
 				)
@@
 		(dnp no)
 		(fields_autoplaced yes)
-		(property "Reference" "#PWR0116"
+		(property "Reference" "#PWR062"
 			(at 161.29 91.44 0)
 			(effects
@@
 			(project "CAN-Interface-Board"
 				(path "/8a3e7f99-4046-40e8-bd7c-d9d1c8c7162e/f33094e5-7720-4bb5-9ddf-b2cfd7a85122"
-					(reference "#PWR0116")
+					(reference "#PWR062")
 					(unit 1)
 				)
@@
 		(dnp no)
 		(fields_autoplaced yes)
-		(property "Reference" "R8"
+		(property "Reference" "R7"
 			(at 163.83 78.7399 0)
 			(effects
@@
 			)
 		)
+		(property "LCSC" "C27834"
+			(at 161.29 80.01 0)
+			(effects
+				(font
+					(size 1.27 1.27)
+				)
+				(hide yes)
+			)
+		)
 		(pin "2"
 		)
@@
 			(project ""
 				(path "/8a3e7f99-4046-40e8-bd7c-d9d1c8c7162e/f33094e5-7720-4bb5-9ddf-b2cfd7a85122"
-					(reference "R8")
-					(unit 1)
-				)
+					(reference "R7")
+					(unit 1)
+				)

Commit message: fixed schematic
Connections:
- net +5V is gone; now on net USB5V: D4.5
- net D+: now also D4.3; no longer D4.1
- net D-: now also D4.1; no longer D4.3
Changed lines of the file:
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@@
 	)
 	(junction
-		(at 110.49 90.17)
+		(at 110.49 91.44)
 		(diameter 0)
 		(color 0 0 0 0)
@@
 	(wire
 		(pts
+			(xy 113.03 90.17) (xy 113.03 87.63)
+		)
+		(stroke
+			(width 0)
+			(type default)
+		)
+	)
+	(wire
+		(pts
 			(xy 78.74 138.43) (xy 82.55 138.43)
 		)
@@
 	(wire
 		(pts
+			(xy 116.84 90.17) (xy 113.03 90.17)
+		)
+		(stroke
+			(width 0)
+			(type default)
+		)
+	)
+	(wire
+		(pts
 			(xy 104.14 85.09) (xy 106.68 85.09)
 		)
@@
 	(wire
 		(pts
-			(xy 110.49 90.17) (xy 116.84 90.17)
+			(xy 114.3 91.44) (xy 110.49 91.44)
 		)
 		(stroke
@@
 	(wire
 		(pts
+			(xy 114.3 87.63) (xy 114.3 91.44)
+		)
+		(stroke
+			(width 0)
+			(type default)
+		)
+	)
+	(wire
+		(pts
 			(xy 106.68 85.09) (xy 110.49 85.09)
 		)
@@
 	(wire
 		(pts
+			(xy 110.49 91.44) (xy 110.49 90.17)
+		)
+		(stroke
+			(width 0)
+			(type default)
+		)
+	)
+	(wire
+		(pts
 			(xy 97.79 83.82) (xy 104.14 83.82)
 		)
@@
 	(wire
 		(pts
-			(xy 106.68 87.63) (xy 116.84 87.63)
-		)
-		(stroke
-			(width 0)
-			(type default)
-		)
-	)
-	(wire
-		(pts
-			(xy 110.49 93.98) (xy 110.49 90.17)
+			(xy 110.49 93.98) (xy 110.49 91.44)
+		)
+		(stroke
+			(width 0)
+			(type default)
+		)
+	)
+	(wire
+		(pts
+			(xy 113.03 87.63) (xy 106.68 87.63)
 		)
 		(stroke
@@
 		(pts
 			(xy 104.14 88.9) (xy 104.14 90.17)
+		)
+		(stroke
+			(width 0)
+			(type default)
+		)
+	)
+	(wire
+		(pts
+			(xy 116.84 87.63) (xy 114.3 87.63)
 		)
 		(stroke
@@
 		(shape output)
 		(at 115.57 71.12 0)
+		(effects
+			(font
+				(size 1.27 1.27)
+			)
+			(justify left)
+		)
+	)
+	(hierarchical_label "USB5V"
+		(shape output)
+		(at 139.7 85.09 0)
 		(effects
 			(font
@@
 	)
 	(symbol
-		(lib_id "power:+5V")
-		(at 139.7 85.09 270)
-		(unit 1)
-		(exclude_from_sim no)
-		(in_bom yes)
-		(on_board yes)
-		(dnp no)
-		(property "Reference" "#PWR060"
-			(at 135.89 85.09 0)
-			(effects
-				(font
-					(size 1.27 1.27)
-				)
-				(hide yes)
-			)
-		)
-		(property "Value" "+5V"
-			(at 143.51 85.0901 90)
-			(effects
-				(font
-					(size 1.27 1.27)
-				)
-				(justify left)
-			)
-		)
-		(property "Footprint" ""
-			(at 139.7 85.09 0)
-			(effects
-				(font
-					(size 1.27 1.27)
-				)
-				(hide yes)
-			)
-		)
-		(property "Datasheet" ""
-			(at 139.7 85.09 0)
-			(effects
-				(font
-					(size 1.27 1.27)
-				)
-				(hide yes)
-			)
-		)
-		(property "Description" "Power symbol creates a global label with name \"+5V\""
-			(at 139.7 85.09 0)
-			(effects
-				(font
-					(size 1.27 1.27)
-				)
-				(hide yes)
-			)
-		)
-		(pin "1"
-		)
-		(instances
-			(project ""
-				(path "/65068a32-f105-4204-b50e-234054c5a6d0/880da092-1c6b-4dcf-a509-490b22fc0ebc"
-					(reference "#PWR052")
-					(unit 1)
-				)
-			)
-			(project "CAN-Interface-Board"
-				(path "/8a3e7f99-4046-40e8-bd7c-d9d1c8c7162e/f33094e5-7720-4bb5-9ddf-b2cfd7a85122"
-					(reference "#PWR060")
-					(unit 1)
-				)
-			)
-		)
-	)
-	(symbol
 		(lib_id "SRV05-4.TCT:SRV05-4.TCT")
 		(at 137.16 87.63 180)
@@
 		(on_board yes)
 		(dnp no)
-		(fields_autoplaced yes)
 		(property "Reference" "D4"
 			(at 127 95.25 0)
@@
 		)
 		(property "Value" "SRV05-4.TCT"
-			(at 127 92.71 0)
+			(at 127.254 96.52 0)
 			(effects
 				(font
@@
 		(lib_id "power:GND")
 		(at 149.86 87.63 0)
+		(mirror y)
 		(unit 1)
 		(exclude_from_sim no)
@@
 		(on_board yes)
 		(dnp no)
-		(fields_autoplaced yes)
 		(property "Reference" "#PWR061"
 			(at 149.86 93.98 0)
